File: dongle.kicad_pcb (KiCad board)
At the start: 2 copper layers, 11.3 x 20.7 mm, 29 parts, among them P1 USB_C_Plug_USB2.0, U1 USBLC6-2P6, U2 nRF52840, Y1 32MHz

Commit message: forgot a silkscreen marker
Other:
- board text added: "SWC"
- board text added: "SWD"
Changed lines of the file:
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@@
   (gr_arc (start 142.844 89.869) (mid 142.463239 90.788239) (end 141.544 91.169)
     (stroke (width 0.1) (type default)) (layer "Edge.Cuts"))
+  (gr_text "SWC" (at 136.764 88.989) (layer "B.SilkS")
+    (effects (font (size 1.5 1.5) (thickness 0.3) bold) (justify left bottom mirror))
+  )
+  (gr_text "SWD" (at 136.764 80.239) (layer "B.SilkS")
+    (effects (font (size 1.5 1.5) (thickness 0.3) bold) (justify left bottom mirror))
+  )
   (segment (start 137.79 85.06761) (end 137.79 84.07) (width 0.13) (layer "F.Cu") (net 1))
   (segment (start 135.06 84.96) (end 135.76 84.96) (width 0.13) (layer "F.Cu") (net 1))
